File: makietadydaktyczna.kicad_pcb (KiCad board)
At the start: 2 copper layers, 148.2 x 77.1 mm, 104 parts, among them J1 Conn_01x06_MountingPin, J10 Conn_01x04_MountingPin, J11 Conn_01x32_MountingPin, J12 Conn_01x05_MountingPin, J13 Conn_01x08_MountingPin, J14 Screw_Terminal_01x08, J15 Conn_01x04_MountingPin, J16 Conn_01x04_MountingPin, J17 Conn_01x02_MountingPin, J2 Conn_01x04_MountingPin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

Commit message: Updated design
-Added multiplexed pins for communication protocols (I2C, UART)
-Fixed problems with ULN2803A COM pin
-Added multiplexed digital pins
-Fixed opamp problems involving disconnected ground plane
-Fixed problem with opamp reading voltage drop from resistor ladder from buttons
-Increased the size of the board a little
Parts:
- removed C19: 100uF, Capacitor_THT:C_Radial_D5.0mm_H11.0mm_P2.00mm
- removed C20: 100nF, Capacitor_SMD:C_0805_2012Metric_Pad1.18x1.45mm_HandSolder
- removed D5: D, SS14:DIOM4325X250N
- removed J13: Conn_01x08_MountingPin, Connector_PinHeader_2.54mm:PinHeader_1x08_P2.54mm_Vertical
- removed the SW8 at (38.0, 70.7)
- added D4: SS14, Diode_SMD:D_SMA, F.Cu at (81.0, 63.0)
- added J18: Screw_Terminal_01x02, TerminalBlock:TerminalBlock_Xinya_XY308-2.54-2P_1x02_P2.54mm_Horizontal, F.Cu at (36.9, 42.2)
- added J19: Conn_01x07, Connector_PinSocket_2.54mm:PinSocket_1x07_P2.54mm_Vertical, F.Cu at (52.8, 63.9)
- added J20: Conn_01x04_MountingPin, Connector_PinSocket_2.54mm:PinSocket_1x04_P2.54mm_Vertical, B.Cu at (49.5, 100.5)
- added J21: Conn_01x04_MountingPin, Connector_PinSocket_2.54mm:PinSocket_1x04_P2.54mm_Vertical, F.Cu at (49.5, 93.0)
- added J22: Conn_01x07, Connector_PinSocket_2.54mm:PinSocket_1x07_P2.54mm_Vertical, F.Cu at (61.0, 41.5)
- added J23: Conn_01x04_MountingPin, Connector_PinSocket_2.54mm:PinSocket_1x04_P2.54mm_Vertical, F.Cu at (36.8, 26.6)
- added J24: Conn_01x04_MountingPin, Connector_PinSocket_2.54mm:PinSocket_1x04_P2.54mm_Vertical, F.Cu at (41.4, 26.6)
- added JP8: Jumper_2_Bridged, Connector_PinHeader_2.54mm:PinHeader_1x02_P2.54mm_Vertical, F.Cu at (47.6, 81.2)
- added SW7: SW_DPST_x2, Button_Switch_THT:SW_PUSH_6mm_H5mm, F.Cu at (116.5, 97.2)
- BZ1, J10, J5, J9: moved to F.Cu
- J15, J16, J2: footprint Connector_PinHeader_2.54mm:PinHeader_1x04_P2.54mm_Vertical -> Connector_PinSocket_2.54mm:PinSocket_1x04_P2.54mm_Vertical
- J17: footprint Connector_PinHeader_2.54mm:PinHeader_1x02_P2.54mm_Vertical -> Connector_PinSocket_2.54mm:PinSocket_1x02_P2.54mm_Vertical
- moved J9 124.4 mm to (160.9, 93.4), turned to -90 degrees
- moved J5 113.1 mm to (160.9, 89.8), turned to -90 degrees
- moved SW2 36.0 mm to (33.5, 87.1)
- moved SW6 12.1 mm to (104.4, 97.2)
- moved SW5 12.1 mm to (92.3, 97.2)
- moved SW4 12.1 mm to (80.2, 97.2)
- moved SW3 12.1 mm to (68.1, 97.2)
- moved BZ1 8.55 mm to (84.4, 49.3), turned to -90 degrees
- moved JP7 5.66 mm to (92.0, 44.1)
- moved SW1 5.54 mm to (33.5, 77.3), turned to 90 degrees
- moved R36 3.10 mm to (87.2, 56.7)
- moved R37 2.90 mm to (89.4, 56.7)
- moved J10 0.10 mm to (49.5, 96.8), turned to -90 degrees
- renumbered RESET to SW8
Connections:
- C14 pad 2: /A3 -> Net-(JP8-B)
- J5 pad 2: GND -> +5V
- J5 pad 3: GND -> /A4/SDA
- J5 pad 4: GND -> /A5/SCL
- J9 pad 2: GND -> +5V
- J9 pad 3: GND -> /A4/SDA
- J9 pad 4: GND -> /A5/SCL
- R2 pad 1: /A3 -> Net-(JP8-B)
- R2 pad 2: Net-(SW8A-B) -> Net-(SW1A-B)
- R26 pad 1: Net-(SW8A-B) -> Net-(SW1A-B)
- R27 pad 1: Net-(SW8A-B) -> Net-(SW1A-B)
- R27 pad 2: Net-(SW1A-B) -> Net-(SW2A-B)
- R28 pad 1: Net-(SW1A-B) -> Net-(SW2A-B)
- R28 pad 2: Net-(SW2A-B) -> Net-(SW3A-B)
- R29 pad 1: Net-(SW2A-B) -> Net-(SW3A-B)
- R29 pad 2: Net-(SW3A-B) -> Net-(SW4A-B)
- R30 pad 1: Net-(SW3A-B) -> Net-(SW4A-B)
- R30 pad 2: Net-(SW4A-B) -> Net-(SW5A-B)
- R31 pad 1: Net-(SW4A-B) -> Net-(SW5A-B)
- R31 pad 2: Net-(SW5A-B) -> Net-(SW6A-B)
- R35 pad 1: Net-(SW5A-B) -> Net-(SW6A-B)
- R35 pad 2: Net-(SW6A-B) -> Net-(SW7A-B)
- U14 pad 10: +5V -> Net-(J18-Pin_1)
Routing:
- net /VIN: track 22.8 -> 70.1 mm, vias 2 -> 3
- net +3.3V: track 51.2 -> 93.8 mm, vias 0 -> 1
- net Net-(SW2A-B): track 47.7 -> 12.1 mm
- net Net-(SW3A-B): track 19.4 -> 47.7 mm
- net /D5: track 105.8 -> 79.9 mm
- net /A0: track 97.7 -> 122.3 mm
- net /D8: track 33.8 -> 56.5 mm
- net Net-(SW1A-B): track 12.1 -> 34.6 mm
- net Net-(SW8A-B): track 21.6 -> 0.00 mm
- net /D9/SPI_CS: track 44.0 -> 23.7 mm
- net /D1/TX: track 22.7 -> 42.8 mm
- net Net-(J18-Pin_1): track 0.00 -> 18.0 mm
- net /D4: track 153.1 -> 135.7 mm
- net /D7: track 158.1 -> 142.6 mm, vias 2 -> 1
- net Net-(SW7A-B): track 0.00 -> 15.4 mm
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Other:
- board size 148.2 x 77.1 mm -> 148.2 x 81.1 mm
- board text removed: "PD2"
- board text removed: "PD3"
- board text removed: "PD4"
- board text removed: "PD5"
- board text removed: "PD7"
- board text removed: "PD9"

Commit message: Add files via upload
Parts:
- BZ1: footprint Buzzer_Beeper:Indicator_PUI_AI-1440-TWT-24V-2-R -> Buzzer_Beeper:Buzzer_D14mm_H7mm_P10mm
- moved Q2 0.81 mm to (86.8, 64.4)
- moved D4 0.50 mm to (81.0, 63.5)
- moved BZ1 0.14 mm to (84.3, 49.4)
- renumbered SW8 to RESET
Routing:
- net /VIN: track 70.1 -> 22.8 mm, vias 3 -> 2
- net +3.3V: track 93.8 -> 51.2 mm, vias 1 -> 0
- net /A0: track 122.3 -> 97.7 mm
- net Net-(SW1A-B): track 34.6 -> 15.2 mm
- net /A2: track 146.3 -> 135.8 mm
- net /A1: track 118.8 -> 108.7 mm
- net GND: track 98.3 -> 105.5 mm
- net Net-(JP7-B): track 3.10 -> 10.2 mm
- net Net-(SW2A-B): track 12.1 -> 14.2 mm
- net Net-(Q2-B): track 11.8 -> 9.92 mm
- net /D5: vias 2 -> 1
- net /D4: vias 3 -> 2
- net /D3: vias 3 -> 2
- net /D2: vias 1 -> 0
Other:
- board text added: "D0"
- board text added: "D1"
- board text added: "D10"
- board text added: "D11"
- board text added: "D12"
- board text added: "D13"
- board text added: "D2"
- board text added: "D3"
- board text added: "D4"
- board text added: "D5"
- board text added: "D6"
- board text added: "D7"
- board text added: "D8"
- board text added: "D9"
