File: makietadydaktyczna.kicad_sch (KiCad schematic)
At the start: 102 parts, among them J1 Conn_01x06_MountingPin, J10 Conn_01x04_MountingPin, J11 Conn_01x32_MountingPin, J12 Conn_01x05_MountingPin, J13 Conn_01x08_MountingPin, J14 Screw_Terminal_01x08, J15 Conn_01x04_MountingPin, J16 Conn_01x04_MountingPin, J17 Conn_01x02_MountingPin, J2 Conn_01x04_MountingPin, J3 Conn_01x16_MountingPin, J4 Conn_01x16_MountingPin, J5 Conn_01x04_MountingPin, J6 Conn_01x05_MountingPin, J7 Conn_01x04_MountingPin, J8 Conn_01x04_MountingPin, J9 Conn_01x04_MountingPin, Q2 Q_NPN_BCE, SW1 SW_DPST_x2, SW2 SW_DPST_x2, SW3 SW_DPST_x2, SW4 SW_DPST_x2, SW5 SW_DPST_x2, SW6 SW_DPST_x2, SW7 SW_DPST_x2, SW8 SW_DPST_x2, U11 TMP36, U13 LM324, U14 ULN2803A, U8 74HC595, U9 74HC595

Commit message: Updated design
-Added multiplexed pins for communication protocols (I2C, UART)
-Fixed problems with ULN2803A COM pin
-Added multiplexed digital pins
-Fixed opamp problems involving disconnected ground plane
-Fixed problem with opamp reading voltage drop from resistor ladder from buttons
-Increased the size of the board a little
Parts:
- removed C19: 100uF, Capacitor_THT:C_Radial_D5.0mm_H11.0mm_P2.00mm, symbol Device:C_Polarized
- removed C20: 100nF, Capacitor_SMD:C_0805_2012Metric_Pad1.18x1.45mm_HandSolder, symbol Device:C
- removed D5: D, SS14:DIOM4325X250N, symbol Device:D
- removed J13: Conn_01x08_MountingPin, symbol Connector_Generic_MountingPin:Conn_01x08_MountingPin
- added D4: SS14, Diode_SMD:D_SMA, symbol Diode:SS14
- added J18: Screw_Terminal_01x02, TerminalBlock:TerminalBlock_Xinya_XY308-2.54-2P_1x02_P2.54mm_Horizontal, symbol Connector:Screw_Terminal_01x02
- added J19, J22: Conn_01x07, Connector_PinSocket_2.54mm:PinSocket_1x07_P2.54mm_Vertical, symbol Connector_Generic:Conn_01x07
- added J20, J21, J23, J24: Conn_01x04_MountingPin, Connector_PinSocket_2.54mm:PinSocket_1x04_P2.54mm_Vertical, symbol Connector_Generic_MountingPin:Conn_01x04_MountingPin
- added JP8: Jumper_2_Bridged, Connector_PinHeader_2.54mm:PinHeader_1x02_P2.54mm_Vertical, symbol Jumper:Jumper_2_Bridged
- J15, J16, J2: footprint Connector_PinHeader_2.54mm:PinHeader_1x04_P2.54mm_Vertical -> Connector_PinSocket_2.54mm:PinSocket_1x04_P2.54mm_Vertical
- J17: footprint Connector_PinHeader_2.54mm:PinHeader_1x02_P2.54mm_Vertical -> Connector_PinSocket_2.54mm:PinSocket_1x02_P2.54mm_Vertical
Connections:
- net +5V: now also J5.2 (Pin_2), J9.2 (Pin_2), D4.1 (K), J20.4 (Pin_4), J21.4 (Pin_4), J23.2 (Pin_2), J24.2 (Pin_2); no longer U14.10
- net A3: now also JP8.1 (A); no longer C14.2, R2.1
- net A4/SDA: now also J5.3 (Pin_3), J9.3 (Pin_3)
- net A4/SDA2: now also J23.3 (Pin_3), J24.3 (Pin_3)
- net A5/SCL: now also J5.4 (Pin_4), J9.4 (Pin_4)
- net A5/SCL2: now also J23.4 (Pin_4), J24.4 (Pin_4)
- net D0/RX/SPI_CS: now also J19.7 (Pin_7)
- net D1/TX: now also J19.6 (Pin_6)
- net D2: now also J19.5 (Pin_5)
- net D3: now also J19.4 (Pin_4), J20.3 (Pin_3), J21.3 (Pin_3)
- net D4: now also J19.3 (Pin_3), J20.2 (Pin_2), J21.2 (Pin_2)
- net D5: now also J19.2 (Pin_2)
- net D6: now also J19.1 (Pin_1)
- net D7: now also J22.7 (Pin_7)
- net D8: now also J22.6 (Pin_6)
- net D9/SPI_CS: now also J22.5 (Pin_5)
- net GND: now also SW8.2 (B), J20.1 (Pin_1), J21.1 (Pin_1), J23.1 (Pin_1), J24.1 (Pin_1); no longer J5.2 (Pin_2), J5.3 (Pin_3), J5.4 (Pin_4), J9.2 (Pin_2), J9.3 (Pin_3), J9.4 (Pin_4), SW8.1 (A)
- net RESET: now also SW8.1 (A); no longer SW7.2 (B)
- net SPI_CS: now also J22.4 (Pin_4)
- net SPI_MISO: now also J22.2 (Pin_2)
- net SPI_MOSI: now also J22.3 (Pin_3)
- net SPI_SCK: now also J22.1 (Pin_1)
- net at R2.2, R26.1, R27.1: now also SW1.2 (B); no longer SW8.2 (B)
- net at R29.2, R30.1: now also SW4.2 (B); no longer SW3.2 (B)
- net at BZ1.2 (-), Q2.2 (C): now also D4.2 (A)
- net at R27.2, R28.1: now also SW2.2 (B); no longer SW1.2 (B)
- net at R28.2, R29.1: now also SW3.2 (B); no longer SW2.2 (B)
- net at R35.2: now also SW7.2 (B); no longer SW6.2 (B)
- net at R30.2, R31.1: now also SW5.2 (B); no longer SW4.2 (B)
- net at R31.2, R35.1: now also SW6.2 (B); no longer SW5.2 (B)
- new net: C14.2, JP8.2 (B), R2.1
- new net: J18.1 (Pin_1), J18.2 (Pin_2), U14.10
Other:
- moved on the sheet: SW8A

Commit message: Add files via upload
Parts:
- BZ1: footprint Buzzer_Beeper:Indicator_PUI_AI-1440-TWT-24V-2-R -> Buzzer_Beeper:Buzzer_D14mm_H7mm_P10mm
Changed lines of the file:
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@@
 			)
 		)
-		(property "Footprint" "Buzzer_Beeper:Indicator_PUI_AI-1440-TWT-24V-2-R"
+		(property "Footprint" "Buzzer_Beeper:Buzzer_D14mm_H7mm_P10mm"
 			(at 116.205 22.86 90)
 			(effects
